File: PCB/C.A.S.E.kicad_pcb (KiCad board)
At the start: 2 copper layers, 34 parts, among them J1 CQ-USB-C16PSMT01, J2 Conn_01x02_Pin, J3 Conn_02x04_Top_Bottom, SW1 SW_Push, SW12 SW_SPDT, SW13 RotaryEncoder_Switch, SW2 SW_Push, SW3 SW_Push, SW4 SW_Push, SW5 SW_Push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

Commit message: adding more stuff
Parts:
- added D1: RED, LED_SMD:LED_0805_2012Metric, F.Cu at (135.2, 132.4)
- added D2: green, LED_SMD:LED_0805_2012Metric, F.Cu at (140.2, 132.4)
- added D3: green, LED_SMD:LED_0805_2012Metric, F.Cu at (130.5, 132.2)
- added G***: LOGO, LOGO, F.Cu at (129.6, 58.1)
- added G***: LOGO, LOGO, B.Cu at (186.4, 156.0)
- added G***: github, All components:github, B.Cu at (183.8, 146.2)
- added G***: LOGO, LOGO, B.Cu at (136.4, 148.2)
- added H1: MountingHole, MountingHole:MountingHole_2.2mm_M2_Pad, F.Cu at (214.9, 155.8)
- added H2: MountingHole, MountingHole:MountingHole_2.2mm_M2_Pad, F.Cu at (118.7, 155.8)
- added H3: MountingHole, MountingHole:MountingHole_2.2mm_M2_Pad, F.Cu at (118.7, 44.7)
- added H4: MountingHole, MountingHole:MountingHole_2.2mm_M2_Pad, F.Cu at (214.9, 44.7)
- added R10: 68, Resistor_SMD:R_1206_3216Metric, B.Cu at (137.3, 137.2)
- added R11: 33, Resistor_SMD:R_1206_3216Metric, B.Cu at (144.2, 132.6)
- added R12: 33, Resistor_SMD:R_1206_3216Metric, B.Cu at (132.1, 137.3)
- added REF**: OSHW-Logo_5.7x6mm_SilkScreen, Symbol:OSHW-Logo_5.7x6mm_SilkScreen, B.Cu at (180.6, 156.4)
- C1, C2, C3, C5, C6, C7, R1, R2, R3, R4, R5, R6, R7, R8, R9: moved to B.Cu
- C4: footprint Capacitor_SMD:C_0201_0603Metric -> Capacitor_SMD:C_1206_3216Metric; moved to B.Cu
- SW12: footprint Button_Switch_THT:SW_CK_JS202011AQN_DPDT_Angled -> All components:SW_JS102011SAQN; moved to B.Cu
- U2: footprint Package_TO_SOT_SMD:SOT-23-5 -> All components:SOT95P285X140-5N; moved to B.Cu
- boot1, rst1: footprint Button_Switch_THT:SW_PUSH_6mm -> All components:SW_PTS645SL43SMTR92LFS; moved to B.Cu
- moved X1 106.3 mm to (130.6, 57.5)
- moved SW12 96.0 mm to (154.9, 41.5)
- moved C4 74.5 mm to (154.6, 56.7), turned to 180 degrees
- moved C1 71.0 mm to (178.7, 67.8)
- moved R5 70.8 mm to (181.8, 60.4), turned to 180 degrees
- moved R4 67.9 mm to (180.3, 56.8), turned to 90 degrees
- moved rst1 65.3 mm to (131.8, 102.3), turned to 180 degrees
- moved boot1 65.0 mm to (142.8, 102.4), turned to 180 degrees
- moved C2 63.9 mm to (172.8, 57.1), turned to 180 degrees
- moved R2 62.1 mm to (174.6, 52.4), turned to 90 degrees
- moved C5 62.1 mm to (168.8, 67.5), turned to 180 degrees
- moved U2 61.7 mm to (173.8, 67.4), turned to 180 degrees
- moved C3 61.2 mm to (168.4, 57.1), turned to 180 degrees
- moved R3 61.2 mm to (172.4, 59.6), turned to 180 degrees
- moved R1 47.6 mm to (159.2, 52.3), turned to -90 degrees
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Connections:
- J3 pad 1: /rst -> /res
- J3 pad 7: VCC -> +3.3V
- U3 pad V: (no net) -> GND
- X1 pad 21: /rst -> /res
Routing:
- net GND: track 0.00 -> 486.6 mm, vias 0 -> 6
- net +3.3V: track 0.00 -> 189.5 mm, vias 0 -> 4
- net /btn_6: track 0.00 -> 104.6 mm, vias 0 -> 2
- net /btn_7: track 0.00 -> 97.2 mm, vias 0 -> 1
- net /IO40: track 0.00 -> 90.9 mm, vias 0 -> 1
- net /btn_4: track 0.00 -> 85.8 mm, vias 0 -> 1
- net /btn_2: track 0.00 -> 82.3 mm, vias 0 -> 1
- net /rst: track 0.00 -> 80.1 mm, vias 0 -> 2
- net /IO39: track 0.00 -> 78.3 mm, vias 0 -> 1
- net /busy: track 0.00 -> 75.6 mm, vias 0 -> 1
- net /IO38: track 0.00 -> 75.3 mm, vias 0 -> 1
- net /dc: track 0.00 -> 71.7 mm, vias 0 -> 1
- net /res: track 0.00 -> 69.8 mm, vias 0 -> 1
- net /btn_1: track 0.00 -> 66.8 mm, vias 0 -> 1
- net /btn_3: track 0.00 -> 64.6 mm, vias 0 -> 1
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Other:
- board outline added: 106.3 x 121.1 mm
- copper layers 2 -> 4
- board text added: "10uF"
- board text added: "33"
- board text added: "68"
- board text added: "boot"
- board text added: "c.a.s.e"
- board text added: "control and shortcut engine"
- board text added: "korV"
- board text added: "made by"
- board text added: "rst"

Commit message: changed everything
Parts:
- removed C3: 4.7uF, LED_SMD:LED_0805_2012Metric
- removed C4: 1uF, Capacitor_SMD:C_1206_3216Metric
- removed C5: 10uF, Capacitor_SMD:C_0805_2012Metric
- removed the G*** at (129.6, 58.1)
- removed the G*** at (186.4, 156.0)
- removed the G*** at (183.8, 146.2)
- removed J2: Conn_01x02_Pin, All components:CONN_S2B-PH-K-S_JST
- removed J3: Conn_02x04_Top_Bottom, Connector_PinHeader_2.54mm:PinHeader_2x04_P2.54mm_Vertical
- removed R3: 3.3k, Resistor_SMD:R_0805_2012Metric
- removed R4: 1.8k, Resistor_SMD:R_1206_3216Metric
- removed R5: 10k, Resistor_SMD:R_0805_2012Metric
- removed R8, R9: 100k, Resistor_SMD:R_1206_3216Metric
- removed REF**: OSHW-Logo_5.7x6mm_SilkScreen, Symbol:OSHW-Logo_5.7x6mm_SilkScreen
- removed SW12: SW_SPDT, All components:SW_JS102011SAQN
- removed U2: AP2112K-3.3, All components:SOT95P285X140-5N
- removed U3: BQ24072TRGTR, All components:RGT16_1P7X1P7
- removed boot1, rst1: SW_Push, All components:SW_PTS645SL43SMTR92LFS
- added ?: LOGO, LOGO, F.Cu at (141.3, 143.9)
- added ?: LOGO, LOGO, F.Cu at (135.1, 147.6)
- added ?: LOGO, LOGO, F.Cu at (135.1, 140.5)
- added ?: LOGO, LOGO, F.Cu at (135.2, 154.7)
- added ?: LOGO, LOGO, F.Cu at (147.3, 147.6)
- added ?: LOGO, LOGO, F.Cu at (122.9, 147.7)
- added ?: LOGO, LOGO, F.Cu at (129.0, 144.0)
- added ?: LOGO, LOGO, F.Cu at (147.3, 140.6)
- added ?: LOGO, LOGO, F.Cu at (141.3, 151.1)
- added ?: LOGO, LOGO, F.Cu at (129.1, 151.2)
- added ?: LOGO, LOGO, F.Cu at (147.5, 154.8)
- added U1: TLV1117-33, All components:SOT230P700X180-4N, B.Cu at (179.6, 148.8)
- added boot: SW_Push, All components:434121025816, B.Cu at (189.3, 101.7)
- added rst: SW_Push, All components:434121025816, B.Cu at (199.4, 101.6)
- C2: value 4.7uF -> 10uF; footprint LED_SMD:LED_0805_2012Metric -> Capacitor_SMD:C_0805_2012Metric
- R1, R2: footprint Resistor_SMD:R_1206_3216Metric -> Resistor_SMD:R_0805_2012Metric
- R10: value 68 -> 150; footprint Resistor_SMD:R_1206_3216Metric -> Resistor_SMD:R_0805_2012Metric
- R11, R12: value 33 -> 150; footprint Resistor_SMD:R_1206_3216Metric -> Resistor_SMD:R_0805_2012Metric
- moved X1 103.8 mm to (194.8, 139.1)
- moved C2 85.8 mm to (178.1, 142.8), turned to -90 degrees
- moved R6 82.1 mm to (206.3, 103.7), turned to -90 degrees
- moved C6 79.9 mm to (206.4, 135.2), turned to -90 degrees
- moved R7 60.6 mm to (210.1, 101.0), turned to -90 degrees
- moved C7 59.9 mm to (206.2, 107.8), turned to 90 degrees
- moved H4 29.6 mm to (208.2, 73.5)
- moved H3 29.2 mm to (122.5, 73.7)
- moved R2 28.1 mm to (156.6, 73.9), turned to -90 degrees
- moved J1 27.2 mm to (164.4, 74.7)
- moved R1 26.4 mm to (174.3, 74.0), turned to 90 degrees
- moved H1 6.82 mm to (208.4, 153.9)
- moved C1 4.74 mm to (174.3, 69.5), turned to 90 degrees
- moved H2 4.30 mm to (122.5, 154.1)
- moved SW3 2.39 mm to (157.9, 119.4)
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Connections:
- C1 pad 1: GND -> VBUS
- C1 pad 2: VBUS -> GND
- C2 pad 1: /VSYS -> +3.3V
- X1 pad 18: /pgood -> unconnected-(X1-IO10-Pad18)
- X1 pad 19: /chg_detection -> unconnected-(X1-IO11-Pad19)
Routing:
- net GND: track 486.6 -> 373.3 mm, vias 6 -> 0
- net VBUS: track 34.7 -> 116.6 mm, vias 3 -> 0
- net /busy: track 75.6 -> 0.00 mm, vias 1 -> 0
- net /dc: track 71.7 -> 0.00 mm, vias 1 -> 0
- net /btn_6: track 104.6 -> 33.6 mm, vias 2 -> 0
- net /res: track 69.8 -> 0.00 mm, vias 1 -> 0
- net /boot: track 47.7 -> 111.0 mm, vias 2 -> 0
- net /btn_7: track 97.2 -> 37.3 mm
- net /cs: track 56.6 -> 0.00 mm, vias 1 -> 0
- net /chg_detection: track 55.4 -> 0.00 mm, vias 2 -> 0
- net /pgood: track 54.0 -> 0.00 mm, vias 2 -> 0
- net /scl: track 53.2 -> 0.00 mm, vias 1 -> 0
- net /sda: track 52.8 -> 0.00 mm, vias 1 -> 0
- net /USB_D-: track 45.6 -> 97.4 mm
- net /VSYS: track 49.1 -> 0.00 mm, vias 2 -> 0
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Other:
- board size 106.3 x 121.1 mm -> 99 x 94.1 mm
- copper layers 4 -> 2
- board text added: "150"
- board text removed: "10uF"
- board text removed: "33"
- board text removed: "68"
- board text removed: "boot"
- board text removed: "control and shortcut engine"
- board text removed: "rst"
