File: PCB/C.A.S.E.kicad_sch (KiCad schematic)
At the start: 34 parts, among them J1 CQ-USB-C16PSMT01, J2 Conn_01x02_Pin, J3 Conn_02x04_Top_Bottom, SW1 SW_Push, SW12 SW_SPDT, SW13 RotaryEncoder_Switch, SW2 SW_Push, SW3 SW_Push, SW4 SW_Push, SW5 SW_Push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

Commit message: adding more stuff
Parts:
- added D1: RED, LED_SMD:LED_0805_2012Metric, symbol Device:LED
- added D2, D3: green, LED_SMD:LED_0805_2012Metric, symbol Device:LED
- added H1, H2, H3, H4: MountingHole, MountingHole:MountingHole_2.2mm_M2_Pad, symbol Mechanical:MountingHole
- added R10: 68, Resistor_SMD:R_1206_3216Metric, symbol Device:R
- added R11, R12: 33, Resistor_SMD:R_1206_3216Metric, symbol Device:R
- C4: footprint Capacitor_SMD:C_0201_0603Metric -> Capacitor_SMD:C_1206_3216Metric
- SW12: footprint Button_Switch_THT:SW_CK_JS202011AQN_DPDT_Angled -> All components:SW_JS102011SAQN
- U2: footprint Package_TO_SOT_SMD:SOT-23-5 -> All components:SOT95P285X140-5N
- boot1, rst1: footprint Button_Switch_THT:SW_PUSH_6mm -> All components:SW_PTS645SL43SMTR92LFS
Connections:
- net VCC is gone; now on net +3.3V: J3.7 (Pin_7)
- net +3.3V: now also R10.2, R11.2, R12.2
- net GND: now also D1.1 (K), D2.1 (K), D3.1 (K)
- net rst: no longer J3.1 (Pin_1), X1.21 (IO13)
- new net: D1.2 (A), R10.1
- new net: D2.2 (A), R11.1
- new net: D3.2 (A), R12.1
- new net res: J3.1 (Pin_1), X1.21 (IO13)

Commit message: changed everything
Parts:
- removed C3: 4.7uF, LED_SMD:LED_0805_2012Metric, symbol Device:C
- removed C4: 1uF, Capacitor_SMD:C_1206_3216Metric, symbol Device:C
- removed C5: 10uF, Capacitor_SMD:C_0805_2012Metric, symbol Device:C
- removed J2: Conn_01x02_Pin, All components:CONN_S2B-PH-K-S_JST, symbol Connector:Conn_01x02_Pin
- removed J3: Conn_02x04_Top_Bottom, Connector_PinHeader_2.54mm:PinHeader_2x04_P2.54mm_Vertical, symbol Connector_Generic:Conn_02x04_Top_Bottom
- removed R3: 3.3k, Resistor_SMD:R_0805_2012Metric, symbol Device:R
- removed R4: 1.8k, Resistor_SMD:R_1206_3216Metric, symbol Device:R
- removed R5: 10k, Resistor_SMD:R_0805_2012Metric, symbol Device:R
- removed R8, R9: 100k, Resistor_SMD:R_1206_3216Metric, symbol Device:R
- removed SW12: SW_SPDT, All components:SW_JS102011SAQN, symbol Switch:SW_SPDT
- removed U2: AP2112K-3.3, All components:SOT95P285X140-5N, symbol Regulator_Linear:AP2112K-3.3
- removed U3: BQ24072TRGTR, All components:RGT16_1P7X1P7, symbol BQ24072TRGTR:BQ24072TRGTR
- added U1: TLV1117-33, All components:SOT230P700X180-4N, symbol Regulator_Linear:TLV1117-33
- C2: value 4.7uF -> 10uF; footprint LED_SMD:LED_0805_2012Metric -> Capacitor_SMD:C_0805_2012Metric
- R1, R2: footprint Resistor_SMD:R_1206_3216Metric -> Resistor_SMD:R_0805_2012Metric
- R10: value 68 -> 150; footprint Resistor_SMD:R_1206_3216Metric -> Resistor_SMD:R_0805_2012Metric
- R11, R12: value 33 -> 150; footprint Resistor_SMD:R_1206_3216Metric -> Resistor_SMD:R_0805_2012Metric
- boot1, rst1: footprint All components:SW_PTS645SL43SMTR92LFS -> All components:434121025816
Connections:
- net VSYS is gone; now on net +3.3V: C2.1
- net +3.3V: now also U1.2 (VO)
- net GND: now also C1.2, U1.1 (GND); no longer C1.1
- net VBUS: now also C1.1, U1.3 (VI); no longer C1.2
- net chg_detection: no longer names the net of X1.19 (IO11)
- net pgood: no longer names the net of X1.18 (IO10)
- no-connect marks 15 -> 17
Other:
- note removed: "jst"
